Commit message: wuyu

File: src/urdf01_rviz/urdf/urdf/demo04_test.urdf (robot description, URDF)
Before this commit: robot my_car, 2 links, 0 joints
Links:
- link base_link: geometry visual cylinder length=0.07 radius=0.30
Joints:
- added joint base_link2base_footprint: type fixed, parent base_footprint, child base_link, origin xyz=0.0 0.0 0.095 rpy=0.0 0.0 0.0, axis 0.0 0.0 0.0

Commit message: model_done

File: src/urdf01_rviz/urdf/urdf/demo04_test.urdf (robot description, URDF)
Before this commit: robot my_car, 2 links, 1 joints
Links:
- added link laser_radar; visual cylinder length=0.04 radius=0.025
- added link wheel_1; visual sphere radius=0.04
- added link wheel_2; visual sphere radius=0.04
- added link wheel_3; visual sphere radius=0.04
- link base_link: geometry visual cylinder length=0.07 radius=0.15
Joints:
- added joint laser_radar2base_link: type fixed, parent base_link, child laser_radar, origin xyz=0.0 0.0 0.055 rpy=0.0 0.0 0.0, axis 0.0 0.0 0.0
- added joint whell_1_to_base_link: type continuous, parent base_link, child wheel_1, origin xyz=-0.14 0.0 -0.055 rpy=0 0.0 0, axis 1 1 0.0
- added joint whell_2_to_base_link: type continuous, parent base_link, child wheel_2, origin xyz=0.07 0.121244 -0.055 rpy=0 0.0 0, axis 1 1 0.0
- added joint whell_3_to_base_link: type continuous, parent base_link, child wheel_3, origin xyz= 0.07 -0.121244 -0.055 rpy=0 0.0 0, axis 1 1 0.0
