Commit message: zuolao

File: src/urdf01_rviz/urdf/urdf/demo03_joint.urdf (robot description, URDF)
Before this commit: robot mycar, 3 links, 2 joints
Links:
- removed link camera
- added link 1_wheel; visual sphere radius=0.04
- added link 2_wheel; visual sphere radius=0.04
- added link 3_wheel; visual sphere radius=0.04
- added link laser_radar; visual cylinder length=0.04 radius=0.025
- link base_link: geometry visual cylinder length=0.07 radius=0.15
Joints:
- removed joint camera2baselink
- added joint 1_wheel2base_link: type continuous, parent base_link, child 1_wheel, origin xyz=-0.14 0 -0.065, axis 1 1 0
- added joint 2_wheel2base_link: type continuous, parent base_link, child 2_wheel, origin xyz=0.07 0.121244 -0.065, axis 1 1 0
- added joint 3_wheel2base_link: type continuous, parent base_link, child 3_wheel, origin xyz=0.07 -0.121244 -0.065, axis 1 1 0
- added joint laser_radar2base_link: type fixed, parent base_link, child laser_radar, origin xyz=0.0 0.0 0.055 rpy=0.0 0.0 0.0, axis 0.0 0.0 0.0
- joint base_link2base_footprint: origin xyz=0 0 0.05 -> xyz=0 0 0.095

Commit message: nice

File: src/urdf01_rviz/urdf/urdf/demo03_joint.urdf (robot description, URDF)
Before this commit: robot my_car, 6 links, 5 joints
Links:
- added link support_laser_radar; visual cylinder length=0.04 radius=0.015
- link laser_radar: geometry visual cylinder length={$ laser_radar_length} radius=0.025
Joints:
- removed joint laser_radar2base_link
- added joint laser_radar2support_laser_radar: type continuous, parent base_link, child laser_radar, origin xyz=0.0 0.0 0.04 rpy=0.0 0.0 0.0, axis 0.0 0.0 1
- added joint support_laser_radar2base_link: type fixed, parent base_link, child support_laser_radar, origin xyz=0.0 0.0 0.055 rpy=0.0 0.0 0.0, axis 0.0 0.0 0.0
- joint 1_wheel2base_link: origin xyz=-0.14 0 -0.065 -> xyz=-0.14 0 -0.055
- joint 2_wheel2base_link: origin xyz=0.07 0.121244 -0.065 -> xyz=0.07 0.121244 -0.055
- joint 3_wheel2base_link: origin xyz=0.07 -0.121244 -0.065 -> xyz=0.07 -0.121244 -0.055

File: src/urdf01_rviz/urdf/xacro/demo01_mycar.xacro (robot description, xacro)
@@ -12,5 +12,5 @@
     <!-- 宏:黑色设置 -->
     <material name="black">
-        <color rgba="0.0 0.0 0.0 1.0" />
+        <color rgba="0.0 0.0 0.0 1" />
     </material>
     <!-- 底盘属性 -->
@@ -33,7 +33,5 @@
         </geometry>
         <origin xyz="0 0 0" rpy="0 0 0" />
-        <material name="black">
-          <color rgba="0 0 0.0 1" />
-        </material>
+        <material name="black"/>
       </visual>
     </link>
@@ -43,22 +41,43 @@
       <origin xyz="0 0 ${earth_space + base_link_length / 2 }" />
     </joint>
-        <!-- Laser Radar link -->
-     <link name="laser_radar">
+    <!-- support_laser -->
+    <xacro:property name="support_laser_radar_length" value="0.04" />
+    <link name="support_laser_radar">
         <visual>
             <origin xyz="0.0 0.0 0.0" rpy="0.0 0.0 0.0"/>
             <geometry>
-                <cylinder radius="0.025" length="0.04"/>
+                <cylinder radius="0.015" length="${support_laser_radar_length }"/>
             </geometry>
-            <material name="laser_radar_color">
-                <color rgba="0.7 0.7 0.7 1.0"/>
+            <material name="support_laser_radar_color">
+                <color rgba="0.1 0.1 0.1 1"/>
             </material>
         </visual>
     </link>
-    <!-- laser_radar2base_link  -->
-    <joint name="laser_radar2base_link" type="fixed">
-        <origin xyz="0.0 0.0 0.055" rpy="0.0 0.0 0.0"/>
+    <!-- support2base_link  -->
+    <joint name="support_laser_radar2base_link" type="fixed">
+        <origin xyz="0.0 0.0 ${base_link_length / 2+support_laser_radar_length / 2}" rpy="0.0 0.0 0.0"/>
         <parent link="base_link"/>
+        <child link="support_laser_radar"/>
+        <axis xyz="0.0 0.0 0.0"/>
+    </joint>
+   <!-- Laser Radar link -->
+   <xacro:property name="laser_radar_length" value="0.04" />
+    <link name="laser_radar">
+        <visual>
+            <origin xyz="0.0 0.0 0.0" rpy="0.0 0.0 0.0"/>
+            <geometry>
+                <cylinder radius="0.025" length="${laser_radar_length}"/>
+            </geometry>
+            <material name="laser_radar_color">
+                <color rgba="0.7 0.7 0.7 1"/>
+            </material>
+        </visual>
+    </link>
+    <!-- laser_radar2support_laser_radar -->
+    <joint name="laser_radar2support_laser_radar" type="continuous">
+        <origin xyz="0.0 0.0 ${laser_radar_length / 2+support_laser_radar_length / 2}" rpy="0.0 0.0 0.0"/>
+        <parent link="support_laser_radar"/>
         <child link="laser_radar"/>
-        <axis xyz="0.0 0.0 0.0"/>
+        <axis xyz="0.0 0.0 1"/>
     </joint>
     <!--wheel link -->
@@ -77,5 +96,5 @@
         </visual>
       </link>
-      <joint name="${name}_wheel2base_link" type="continuous">
+      <joint name="base_${name}_wheel_joint" type="continuous">
           <parent link="base_link" />
           <child link="${name}_wheel" />
@@ -84,6 +103,6 @@
       </joint>
     </xacro:macro>
-    <xacro:add_wheel name="1" flag1="-0.14" flag2="0"/>
-    <xacro:add_wheel name="2" flag1="0.07" flag2="0.121244"/>
-    <xacro:add_wheel name="3" flag1="0.07" flag2="-0.121244"/>
+    <xacro:add_wheel name="l" flag1="-0.14" flag2="0"/>
+    <xacro:add_wheel name="r" flag1="0.07" flag2="0.121244"/>
+    <xacro:add_wheel name="b" flag1="0.07" flag2="-0.121244"/>
 </robot>
