Commit message: car over

File: src/urdf02_gazebo/urdf/mycar.xacro (robot description, xacro)
@@ -152,6 +152,6 @@
     <!-- 摄像头属性 -->
     <xacro:property name="camera_length" value="0.01" /> <!-- 摄像头长度(x) -->
-    <xacro:property name="camera_width" value="0.025" /> <!-- 摄像头宽度(y) -->
-    <xacro:property name="camera_height" value="0.025" /> <!-- 摄像头高度(z) -->
+    <xacro:property name="camera_width" value="0.045" /> <!-- 摄像头宽度(y) -->
+    <xacro:property name="camera_height" value="0.035" /> <!-- 摄像头高度(z) -->
     <xacro:property name="camera_x" value="0.10" /> <!-- 摄像头安装的x坐标 -->
     <xacro:property name="camera_y" value="0.0" /> <!-- 摄像头安装的y坐标 -->

Commit message: yaosi

File: src/urdf02_gazebo/urdf/mycar.xacro (robot description, xacro)
@@ -19,5 +19,5 @@
     <xacro:property name="base_link_radius" value="0.15" /> <!-- base_link 半径 -->
     <xacro:property name="base_link_length" value="0.07" /> <!-- base_link 长 -->
-    <xacro:property name="base_link_weight" value="2" />
+    <xacro:property name="base_link_weight" value="3" />
     <xacro:property name="earth_space" value="0.06" /> <!-- 离地间距 -->
     <!-- 底盘 -->
@@ -72,5 +72,5 @@
             </geometry>
         </collision>
-        <xacro:cylinder_inertial_matrix m="0.05"  r="0.015" h="${support_laser_radar_length }" />
+        <xacro:cylinder_inertial_matrix m="0.5"  r="0.015" h="${support_laser_radar_length }" />
     </link>
     <gazebo reference="support_laser_radar">
@@ -102,5 +102,5 @@
             </geometry>
         </collision>
-        <xacro:cylinder_inertial_matrix m="0.1"  r="0.025" h="${laser_radar_length}" />
+        <xacro:cylinder_inertial_matrix m="0.2"  r="0.025" h="${laser_radar_length}" />
     </link>
     <gazebo reference="laser_radar">
@@ -115,7 +115,7 @@
     </joint>
     <!--wheel link -->
-     <xacro:property name="wheel_radius" value="0.04" /> <!-- 支撑轮半径 -->
+     <xacro:property name="wheel_radius" value="0.04" /> <!-- 轮半径 -->
     <!-- wheel宏 -->
-    <xacro:macro name="add_wheel" params="name flag1 flag2" >
+    <xacro:macro name="add_wheel" params="name flag1 flag2 zyd_x zyd_y zyd_z" >
       <link name="${name}_wheel">
         <visual>
@@ -143,10 +143,11 @@
           <child link="${name}_wheel" />
           <origin xyz="${flag1} ${flag2} ${-(base_link_length / 2 + earth_space / 2)+0.01}" />
-          <axis xyz="1 1 0" />
+          <axis xyz="${zyd_x} ${zyd_y} ${zyd_z}" />
+          <dynamics damping="0.4" friction="1.0"/>
       </joint>
     </xacro:macro>
-    <xacro:add_wheel name="l" flag1="-0.14" flag2="0"/>
-    <xacro:add_wheel name="r" flag1="0.07" flag2="0.121244"/>
-    <xacro:add_wheel name="b" flag1="0.07" flag2="-0.121244"/>
+    <xacro:add_wheel name="l" flag1="-0.14" flag2="0"  zyd_x="1" zyd_y="1" zyd_z="0"/>
+    <xacro:add_wheel name="r" flag1="0.07" flag2="0.121244" zyd_x="1" zyd_y="1" zyd_z="0"/>
+    <xacro:add_wheel name="b" flag1="0.07" flag2="-0.121244" zyd_x="1" zyd_y="1" zyd_z="0"/>
     <!-- 摄像头相关的 xacro 文件 -->
     <!-- 摄像头属性 -->
@@ -183,3 +184,6 @@
         <material>Gazebo/Grey</material>
     </gazebo>
+    <xacro:include filename="gazebo/move.xacro"/>
+    <xacro:include filename="gazebo/laser.xacro"/>
+    <xacro:include filename="gazebo/camera.xacro"/>
 </robot>
